Commit message: fixed wrong wstool path install, switched hotspray_ur5_moveit package with plane original ur5_moveit package, some minor changes

File: hotspray_ur5_description/urdf/hotspray_ur5_demo.urdf.xacro (robot description, xacro)
@@ -2,17 +2,30 @@
 <robot xmlns:xacro="http://www.ros.org/wiki/xacro" name="hotspray_ur5_description">
   <!--  <xacro:include filename="$(find ur5_support)/urdf/ur5_macro.xacro"/> -->
-  <xacro:include filename="$(find ur_description)/urdf/ur5_joint_limited_robot.urdf.xacro"/>
+  <!-- xacro:include filename="$(find ur_description)/urdf/ur5_joint_limited_robot.urdf.xacro"/-->
   <xacro:include filename="$(find hotspray_ur5_description)/urdf/hotspray_tool.urdf.xacro"/>
   <xacro:include filename="$(find hotspray_ur5_description)/urdf/ur5_table.urdf.xacro"/>
   <xacro:property name="prefix" value=""/>
   <!-- robot -->
-  <link name="world_frame"/>
-  <joint name="world_to_baselink" type="fixed">
-    <parent link="world_frame"/>
-    <child link="base_link"/>
-    <origin  xyz="0 0 0.05" rpy="0 0 0" />
-  </joint>
-  <!-- robot
-  <xacro:ur5_robot prefix="${prefix}"/> -->
+  <xacro:arg name="transmission_hw_interface" default="hardware_interface/PositionJointInterface"/>
+    <!-- common stuff -->
+    <xacro:include filename="$(find ur_description)/urdf/common.gazebo.xacro" />
+    <!-- ur5 -->
+    <xacro:include filename="$(find ur_description)/urdf/ur5.urdf.xacro" />
+    <!-- arm -->
+    <xacro:ur5_robot prefix="${prefix}" joint_limited="true"
+      shoulder_pan_lower_limit="${-pi}" shoulder_pan_upper_limit="${pi}"
+      shoulder_lift_lower_limit="${-pi}" shoulder_lift_upper_limit="${pi}"
+      elbow_joint_lower_limit="${-pi}" elbow_joint_upper_limit="${pi}"
+      wrist_1_lower_limit="${-pi}" wrist_1_upper_limit="${pi}"
+      wrist_2_lower_limit="${-pi}" wrist_2_upper_limit="${pi}"
+      wrist_3_lower_limit="${-pi}" wrist_3_upper_limit="${pi}"
+      transmission_hw_interface="$(arg transmission_hw_interface)"
+    />
+    <link name="world_frame"/>
+    <joint name="world_to_baselink" type="fixed">
+      <parent link="world_frame"/>
+      <child link="base_link"/>
+      <origin  xyz="0 0 0.05" rpy="0 0 0" />
+    </joint>
   <!-- table -->
   <xacro:table parent="world_frame">
