Commit message: fixed robot simulation, loading joint names from seperate file

File: hotspray_ur5_description/urdf/hotspray_extruder.urdf.xacro (robot description, xacro)
@@ -18,10 +18,10 @@
         </material>
       </visual>
-      <collision>
+      <!--collision>
         <origin xyz="0.04 -0.06 0.06" rpy="${-pi/2} ${-pi/2} ${pi/2}" />
         <geometry>
           <box size="0.195 0.04 0.27"/>
         </geometry>
-      </collision>
+      </collision-->
     </link>
     <!--joint between fixture and hotspray-->

File: hotspray_ur5_description/urdf/hotspray_ur5_demo.urdf.xacro (robot description, xacro)
@@ -5,4 +5,6 @@
   <xacro:include filename="$(find hotspray_ur5_description)/urdf/hotspray_tool.urdf.xacro"/>
   <xacro:include filename="$(find hotspray_ur5_description)/urdf/ur5_table.urdf.xacro"/>
+    <!-- ur5 -->
+    <xacro:include filename="$(find ur_description)/urdf/ur5.urdf.xacro" />
   <xacro:property name="prefix" value=""/>
   <!-- robot -->
@@ -10,6 +12,4 @@
     <!-- common stuff -->
     <xacro:include filename="$(find ur_description)/urdf/common.gazebo.xacro" />
-    <!-- ur5 -->
-    <xacro:include filename="$(find ur_description)/urdf/ur5.urdf.xacro" />
     <!-- arm -->
     <xacro:ur5_robot prefix="${prefix}" joint_limited="true"

File: hotspray_ur5_description/urdf/ur5_table.urdf.xacro (robot description, xacro)
@@ -14,10 +14,10 @@
     <xacro:macro name="table" params="parent *origin">
     <link name="table">
-        <collision><!-- bottom -->
+        <!--collision>< bottom >
           <origin rpy="0 0 0" xyz="-0.2 -0.2 0.025"/>
           <geometry>
              <box size="${workspace_x} ${workspace_y} ${wall_width}"/>
           </geometry>
-        </collision>
+        </collision-->
         <visual>
           <origin rpy="0 0 0" xyz="-0.2 -0.2 0.025"/>
